File: wifi-multimeter-pcb/power.sch (KiCad schematic (older format))
At the start: 13 parts, among them J2 USB_B_Micro, J3 Conn_01x02, U2 AMS1117-3.3, U3 LTC4054ES5-4.2

Commit message: update pcb
Parts:
- J3: value Conn_01x02 -> BATT
Connections:
- wire segments 30 -> 29
Changed lines of the file:
@@
 $Descr A4 11693 8268
 encoding utf-8
-Sheet 2 2
+Sheet 2 4
 Title "power"
 Date "2020-07-26"
@@
 AR Path="/5F232336" Ref="J?"  Part="1"
 AR Path="/5F2186C0/5F232336" Ref="J3"  Part="1"
-F 0 "J3" H 6368 2475 50  0000 C CNN
-F 1 "Conn_01x02" H 6368 2566 50  0000 C CNN
+F 0 "J3" H 6450 2600 50  0000 C CNN
+F 1 "BATT" H 6450 2900 50  0000 C CNN
 F 2 "Connector_PinHeader_2.54mm:PinHeader_1x02_P2.54mm_Vertical" H 6450 2800 50  0001 C CNN
 F 3 "~" H 6450 2800 50  0001 C CNN
@@
 AR Path="/5F2186C0/5F24A06E" Ref="#PWR012"  Part="1"
 F 0 "#PWR012" H 4200 3750 50  0001 C CNN
-F 1 "+3.3V" H 4215 4073 50  0000 C CNN
+F 1 "+3.3V" V 4200 4150 50  0000 C CNN
 F 2 "" H 4200 3900 50  0001 C CNN
 F 3 "" H 4200 3900 50  0001 C CNN
@@
 	3200 3900 3050 3900
 Connection ~ 3050 3900
-Wire Wire Line
-	3050 3750 3050 3900
 NoConn ~ 3350 2700
 NoConn ~ 3350 2800
